File: hardware/kicad/PDU.kicad_sch (KiCad schematic)
At the start: 12 parts, among them IC1 AP64352QSP-13

Commit message: added 3.3v
Parts:
- added C10, C8: 10uF, Capacitor_SMD:C_0603_1608Metric_Pad1.08x0.95mm_HandSolder, symbol Device:C
- added C11, C12, C13, C14, C9: 100nF, Capacitor_SMD:C_0603_1608Metric_Pad1.08x0.95mm_HandSolder, symbol Device:C
- added D1, D3: LED, LED_SMD:LED_0805_2012Metric_Pad1.15x1.40mm_HandSolder, symbol 2026-06-29_10-35-29:LED
- added D2: VS3V3BA1EST15R, VS3V3BA1EST15R, symbol SamacSys_Parts:VS3V3BA1EST15R
- added FB1: BLM21PG300SN1D, BEADC2012X105N, symbol SamacSys_Parts:BLM21PG300SN1D
- added IC2: AP7363-33D-13, AP736333D13, symbol SamacSys_Parts:AP7363-33D-13
- added IC3: INA181A2QDBVRQ1, SOT95P280X145-6N, symbol SamacSys_Parts:INA181A2QDBVRQ1
- added R4, R7: 4.7k, Resistor_SMD:R_0603_1608Metric_Pad0.98x0.95mm_HandSolder, symbol Device:R
- added R5: 1M, Resistor_SMD:R_0603_1608Metric_Pad0.98x0.95mm_HandSolder, symbol Device:R
- added R6, R8: 100k, Resistor_SMD:R_0603_1608Metric_Pad0.98x0.95mm_HandSolder, symbol Device:R
Connections:
- net +24V: now also R5.1
- net +5V: now also C14.2, C8.1, C9.2, IC2.1 (IN), IC3.6 (VS), R7.1
- net GND: now also C5.2, C6.2, C7.2, R3.2, C10.2, C11.1, C12.2, C13.1, C14.1, C8.2, C9.1, D1.1 (K), D2.1, D3.1 (K), IC3.2 (GND), IC3.5 (REF), R6.1
- new net: D3.2 (A), R7.2
- new net: D1.2 (A), R4.2
- new net: C12.1, D2.2, R5.2, R6.2
- new net: IC3.1 (OUT), R8.1
- new net: FB1.1, IC2.3 (OUT)
- new net +3V3: C10.1, C11.2, FB1.2, R4.1
- new net CURRENT_ADC: C13.2, R8.2
- new net SHUNT_IN: IC3.3 (IN+)
- new net SHUNT_OUT: IC3.4 (IN-)
Other:
- moved on the sheet: C1, C2, C3, C4, C5, C6, C7, IC1, L1, R1, R2, R3
