File: hardware/kicad/vajran.kicad_pcb (KiCad board)
At the start: 2 copper layers, 0 parts

Commit message: added 24v to 5v
Parts:
- added C1: 10uF, Capacitor_SMD:C_0603_1608Metric_Pad1.08x0.95mm_HandSolder, F.Cu at (63.9, 47.4)
- added C2: 100nF, Capacitor_SMD:C_0603_1608Metric_Pad1.08x0.95mm_HandSolder, F.Cu at (63.9, 49.9)
- added C3: 10uF, Capacitor_SMD:C_0603_1608Metric_Pad1.08x0.95mm_HandSolder, F.Cu at (63.9, 52.4)
- added C4: 100nF, Capacitor_SMD:C_0603_1608Metric_Pad1.08x0.95mm_HandSolder, F.Cu at (63.9, 55.0)
- added C5: 10nF, Capacitor_SMD:C_0603_1608Metric_Pad1.08x0.95mm_HandSolder, F.Cu at (63.9, 57.5)
- added C6: 22uF, Capacitor_SMD:C_0603_1608Metric_Pad1.08x0.95mm_HandSolder, F.Cu at (63.9, 60.0)
- added C7: 22uf, Capacitor_SMD:C_0603_1608Metric_Pad1.08x0.95mm_HandSolder, F.Cu at (63.9, 62.5)
- added IC1: AP64352QSP-13, AP64352QSP-13:SOIC127P600X163-9N, F.Cu at (70.3, 59.0)
- added L1: SRP5030HMCT-5R6M, SRP5030HMCT-5R6M:SRP5030HMCT100M, F.Cu at (69.8, 51.0)
- added R1: 200k, Resistor_SMD:R_0603_1608Metric_Pad0.98x0.95mm_HandSolder, F.Cu at (63.9, 65.0)
- added R2: 115k, Resistor_SMD:R_0603_1608Metric_Pad0.98x0.95mm_HandSolder, F.Cu at (63.9, 67.5)
- added R3: 22.1k, Resistor_SMD:R_0603_1608Metric_Pad0.98x0.95mm_HandSolder, F.Cu at (63.9, 70.0)

Commit message: updated
Parts:
- added C10: 10uF, Capacitor_SMD:C_0603_1608Metric_Pad1.08x0.95mm_HandSolder, F.Cu at (26.2, 48.5)
- added C11: 100nF, Capacitor_SMD:C_0603_1608Metric_Pad1.08x0.95mm_HandSolder, F.Cu at (26.2, 51.0)
- added C12: 100nF, Capacitor_SMD:C_0603_1608Metric_Pad1.08x0.95mm_HandSolder, F.Cu at (30.6, 43.5)
- added C13: 100nF, Capacitor_SMD:C_0603_1608Metric_Pad1.08x0.95mm_HandSolder, F.Cu at (30.6, 46.0)
- added C14: 100nF, Capacitor_SMD:C_0603_1608Metric_Pad1.08x0.95mm_HandSolder, F.Cu at (30.6, 48.5)
- added C15: 22uF, Capacitor_SMD:C_0603_1608Metric_Pad1.08x0.95mm_HandSolder, F.Cu at (44.7, 43.5)
- added C16: 10uF, Capacitor_SMD:C_0603_1608Metric_Pad1.08x0.95mm_HandSolder, F.Cu at (44.7, 46.0)
- added C17: 100nF, Capacitor_SMD:C_0603_1608Metric_Pad1.08x0.95mm_HandSolder, F.Cu at (44.7, 48.5)
- added C8: 10uF, Capacitor_SMD:C_0603_1608Metric_Pad1.08x0.95mm_HandSolder, F.Cu at (26.2, 43.5)
- added C9: 100nF, Capacitor_SMD:C_0603_1608Metric_Pad1.08x0.95mm_HandSolder, F.Cu at (26.2, 46.0)
- added D1: LED, LED_SMD:LED_0805_2012Metric_Pad1.15x1.40mm_HandSolder, F.Cu at (36.2, 58.4)
- added D2: VS3V3BA1EST15R, SamacSys_Parts:VS3V3BA1EST15R, F.Cu at (38.8, 44.1)
- added D3: LED, LED_SMD:LED_0805_2012Metric_Pad1.15x1.40mm_HandSolder, F.Cu at (36.2, 61.4)
- added D4: CDSOT23-SM712, SamacSys_Parts:SOT95P230X117-3N, F.Cu at (49.3, 51.0)
- added FB1: BLM21PG300SN1D, SamacSys_Parts:BEADC2012X105N, F.Cu at (36.0, 64.5)
- added IC2: AP7363-33D-13, SamacSys_Parts:AP736333D13, F.Cu at (28.9, 59.0)
- added IC3: INA181A2QDBVRQ1, SamacSys_Parts:SOT95P280X145-6N, F.Cu at (36.4, 54.6)
- added IC4: THVD1500DR, SamacSys_Parts:SOIC127P600X175-8N, F.Cu at (51.1, 45.5)
- added R10: 120R, Resistor_SMD:R_0603_1608Metric_Pad0.98x0.95mm_HandSolder, F.Cu at (44.7, 53.5)
- added R11: 4.7k, Resistor_SMD:R_0603_1608Metric_Pad0.98x0.95mm_HandSolder, F.Cu at (44.7, 56.0)
- added R12: 4.7k, Resistor_SMD:R_0603_1608Metric_Pad0.98x0.95mm_HandSolder, F.Cu at (44.7, 58.5)
- added R13: 10R, Resistor_SMD:R_0603_1608Metric_Pad0.98x0.95mm_HandSolder, F.Cu at (44.7, 61.0)
- added R14: 10R, Resistor_SMD:R_0603_1608Metric_Pad0.98x0.95mm_HandSolder, F.Cu at (44.7, 63.6)
- added R4: 4.7k, Resistor_SMD:R_0603_1608Metric_Pad0.98x0.95mm_HandSolder, F.Cu at (30.6, 51.0)
- added R5: 1M, Resistor_SMD:R_0603_1608Metric_Pad0.98x0.95mm_HandSolder, F.Cu at (34.9, 43.5)
- added R6: 100k, Resistor_SMD:R_0603_1608Metric_Pad0.98x0.95mm_HandSolder, F.Cu at (34.9, 46.0)
- added R7: 4.7k, Resistor_SMD:R_0603_1608Metric_Pad0.98x0.95mm_HandSolder, F.Cu at (34.9, 48.5)
- added R8: 100k, Resistor_SMD:R_0603_1608Metric_Pad0.98x0.95mm_HandSolder, F.Cu at (34.9, 51.0)
- added R9: 4.7k, Resistor_SMD:R_0603_1608Metric_Pad0.98x0.95mm_HandSolder, F.Cu at (44.7, 51.0)
- moved L1 9.34 mm to (78.1, 46.7)
Connections:
- C5 pad 2: Net-(C5-Pad2) -> GND
- C6 pad 2: Net-(C5-Pad2) -> GND
- C7 pad 2: Net-(C5-Pad2) -> GND
- R3 pad 2: Net-(C5-Pad2) -> GND
Other:
- board outline added: 71.8 x 51.4 mm
- copper layers 2 -> 4
